File: Hardware/RevA/KiCad/SimonShield.kicad_pcb (KiCad board)
At the start: 2 copper layers, 68.6 x 53.3 mm, 40 parts, among them J1 ARDUINO, SW0 LED_KEY, SW1 LED_KEY, SW2 LED_KEY, SW3 LED_KEY

Commit message: exchanged buzzer footprint
Parts:
- added VIA: GND, via, F.Cu at (174.4, 101.0)
- moved VIA 8.13 mm to (170.4, 93.9)
Routing:
- net +5V: track 70.5 -> 64.5 mm
- net /BZ0_B: track 80.0 -> 84.8 mm
- net Net-(BZ0-Pad1): track 9.42 -> 12.0 mm
Changed lines of the file:
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@@
 (kicad_pcb (version 4) (host pcbnew 4.0.7)
   (general
-    (links 62)
+    (links 65)
     (no_connects 0)
     (area 115.179499 78.349499 184.540501 132.470501)
     (thickness 1.6)
     (drawings 31)
-    (tracks 103)
+    (tracks 105)
     (zones 0)
-    (modules 40)
+    (modules 41)
     (nets 37)
   )
@@
     (34 B.Paste user)
     (35 F.Paste user)
-    (36 B.SilkS user)
-    (37 F.SilkS user hide)
+    (36 B.SilkS user hide)
+    (37 F.SilkS user)
     (38 B.Mask user)
     (39 F.Mask user)
@@
   )
   (module via (layer F.Cu)
+    (at 174.371 100.965)
+    (fp_text reference VIA (at 0 0.7) (layer F.SilkS) hide
+      (effects (font (size 0.5 0.5) (thickness 0.125)))
+    )
+    (fp_text value GND (at 0 -0.7) (layer F.SilkS) hide
+      (effects (font (size 0.5 0.5) (thickness 0.125)))
+    )
+    (pad "" thru_hole circle (at 0 0) (size 0.62 0.62) (drill 0.4) (layers *.Cu)
+      (net 18 GND) (zone_connect 2))
+  )
+  (module via (layer F.Cu)
+    (at 170.053 97.79)
+    (fp_text reference VIA (at 0 0.7) (layer F.SilkS) hide
+      (effects (font (size 0.5 0.5) (thickness 0.125)))
+    )
+    (fp_text value GND (at 0 -0.7) (layer F.SilkS) hide
+      (effects (font (size 0.5 0.5) (thickness 0.125)))
+    )
+    (pad "" thru_hole circle (at 0 0) (size 0.62 0.62) (drill 0.4) (layers *.Cu)
+      (net 18 GND) (zone_connect 2))
+  )
+  (module buzzer (layer F.Cu)
+    (at 176.53 86.36)
+    (descr Buzzer)
+    (tags buzzer)
+    (autoplace_cost180 10)
+    (fp_text reference BZ0 (at 0 0) (layer F.SilkS)
+      (effects (font (size 0.99822 0.99822) (thickness 0.19812)))
+    )
+    (fp_text value BUZZER (at 0 -5.969) (layer F.SilkS) hide
+      (effects (font (size 0.99822 0.99822) (thickness 0.19812)))
+    )
+    (fp_circle (center 0 0) (end 5.08 -1.27) (layer F.SilkS) (width 0.15))
+    (pad 1 thru_hole circle (at 0 3.175) (size 2 2) (drill 1) (layers *.Cu *.Mask)
+      (net 36 "Net-(BZ0-Pad1)"))
+    (pad 2 thru_hole circle (at 0 -3.175) (size 2 2) (drill 1) (layers *.Cu *.Mask)
+      (net 27 /BZ0_B))
+    (pad 2 thru_hole circle (at -2.54 0) (size 2 2) (drill 1) (layers *.Cu *.Mask)
+      (net 27 /BZ0_B))
+    (pad 1 thru_hole circle (at 2.54 0) (size 2 2) (drill 1) (layers *.Cu *.Mask)
+      (net 36 "Net-(BZ0-Pad1)"))
+    (model ${KIPRJMOD}/3D-Models/buzzer.wrl
+      (at (xyz 0 0 0))
+      (scale (xyz 1 1 1))
+      (rotate (xyz 0 0 0))
+    )
+  )
+  (module via (layer F.Cu)
     (at 147.701 127.254)
     (fp_text reference VIA (at 0 0.7) (layer F.SilkS) hide
@@
   )
   (module via (layer F.Cu)
-    (at 170.053 97.79)
-    (fp_text reference VIA (at 0 0.7) (layer F.SilkS) hide
-      (effects (font (size 0.5 0.5) (thickness 0.125)))
-    )
-    (fp_text value GND (at 0 -0.7) (layer F.SilkS) hide
-      (effects (font (size 0.5 0.5) (thickness 0.125)))
-    )
-    (pad "" thru_hole circle (at 0 0) (size 0.62 0.62) (drill 0.4) (layers *.Cu)
-      (net 18 GND) (zone_connect 2))
-  )
-  (module via (layer F.Cu)
-    (at 174.371 100.965)
+    (at 170.434 93.853)
     (fp_text reference VIA (at 0 0.7) (layer F.SilkS) hide
       (effects (font (size 0.5 0.5) (thickness 0.125)))
@@
     (model ${KIPRJMOD}/3D-Models/arduino_top_header.wrl
       (at (xyz 0 0 -0.07000000000000001))
-      (scale (xyz 1 1 1))
-      (rotate (xyz 0 0 0))
-    )
-  )
-  (module buzzer (layer F.Cu)
-    (at 176.53 86.36)
-    (descr Buzzer)
-    (tags buzzer)
-    (autoplace_cost180 10)
-    (fp_text reference BZ0 (at 0 0) (layer F.SilkS)
-      (effects (font (size 0.99822 0.99822) (thickness 0.19812)))
-    )
-    (fp_text value BUZZER (at 0 2) (layer F.SilkS) hide
-      (effects (font (size 0.99822 0.99822) (thickness 0.19812)))
-    )
-    (fp_circle (center 0 0) (end 5.08 -1.27) (layer F.SilkS) (width 0.15))
-    (pad 2 thru_hole circle (at -3.8 0) (size 2 2) (drill 1) (layers *.Cu *.Mask)
-      (net 27 /BZ0_B))
-    (pad 1 thru_hole circle (at 3.8 0) (size 2 2) (drill 1) (layers *.Cu *.Mask)
-      (net 36 "Net-(BZ0-Pad1)"))
-    (model ${KIPRJMOD}/3D-Models/buzzer.wrl
-      (at (xyz 0 0 0))
       (scale (xyz 1 1 1))
       (rotate (xyz 0 0 0))
@@
   (gr_circle (center 146.05 105.41) (end 146.05 114.3) (layer F.SilkS) (width 1))
   (gr_circle (center 146.05 105.41) (end 146.05 127.635) (layer F.SilkS) (width 1))
-  (segment (start 181.61 100.33) (end 177.8 96.52) (width 0.6) (layer B.Cu) (net 17))
-  (segment (start 146.05 82.55) (end 146.05 81.28) (width 0.6) (layer B.Cu) (net 17) (status 20))
-  (segment (start 147.32 83.82) (end 146.05 82.55) (width 0.6) (layer B.Cu) (net 17))
-  (segment (start 175.26 83.82) (end 147.32 83.82) (width 0.6) (layer B.Cu) (net 17))
-  (segment (start 177.8 86.36) (end 175.26 83.82) (width 0.6) (layer B.Cu) (net 17))
-  (segment (start 177.8 96.52) (end 177.8 86.36) (width 0.6) (layer B.Cu) (net 17))
+  (segment (start 181.61 100.33) (end 165.1 83.82) (width 0.6) (layer F.Cu) (net 17))
+  (segment (start 146.05 82.55) (end 146.05 81.28) (width 0.6) (layer F.Cu) (net 17))
+  (segment (start 147.32 83.82) (end 146.05 82.55) (width 0.6) (layer F.Cu) (net 17))
+  (segment (start 165.1 83.82) (end 147.32 83.82) (width 0.6) (layer F.Cu) (net 17))
   (segment (start 181.61 120.65) (end 181.61 115.57) (width 0.6) (layer F.Cu) (net 17))
   (segment (start 181.61 115.57) (end 181.61 110.49) (width 0.6) (layer F.Cu) (net 17))
@@
   (segment (start 138.43 128.905) (end 141.605 125.73) (width 0.3) (layer B.Cu) (net 26) (status 10))
   (segment (start 141.605 125.73) (end 161.29 125.73) (width 0.3) (layer B.Cu) (net 26))
-  (segment (start 179.07 123.19) (end 175.895 126.365) (width 0.3) (layer B.Cu) (net 27))
-  (segment (start 172.73 86.36) (end 169.545 89.545) (width 0.3) (layer B.Cu) (net 27))
+  (segment (start 173.99 86.36) (end 176.53 83.82) (width 0.3) (layer B.Cu) (net 27))
+  (segment (start 176.53 83.82) (end 176.53 83.185) (width 0.3) (layer B.Cu) (net 27))
+  (segment (start 169.545 95.885) (end 169.545 90.805) (width 0.3) (layer B.Cu) (net 27))
   (segment (start 179.07 104.14) (end 179.07 106.68) (width 0.3) (layer B.Cu) (net 27))
   (segment (start 172.085 97.155) (end 179.07 104.14) (width 0.3) (layer B.Cu) (net 27))
   (segment (start 170.815 97.155) (end 172.085 97.155) (width 0.3) (layer B.Cu) (net 27))
   (segment (start 169.545 95.885) (end 170.815 97.155) (width 0.3) (layer B.Cu) (net 27))
-  (segment (start 169.545 89.545) (end 169.545 95.885) (width 0.3) (layer B.Cu) (net 27))
   (segment (start 179.07 106.68) (end 179.07 123.19) (width 0.3) (layer B.Cu) (net 27))
-  (segment (start 147.32 126.365) (end 145.034 128.651) (width 0.3) (layer B.Cu) (net 27) (status 20))
+  (segment (start 145.034 128.651) (end 147.32 126.365) (width 0.3) (layer B.Cu) (net 27) (status 20))
   (segment (start 175.895 126.365) (end 147.32 126.365) (width 0.3) (layer B.Cu) (net 27))
+  (segment (start 179.07 123.19) (end 175.895 126.365) (width 0.3) (layer B.Cu) (net 27))
+  (segment (start 169.545 90.805) (end 173.99 86.36) (width 0.3) (layer B.Cu) (net 27))
   (segment (start 145.034 128.651) (end 145.034 129.54) (width 0.3) (layer B.Cu) (net 27) (status 30))
   (segment (start 147.574 129.54) (end 147.574 128.651) (width 0.3) (layer B.Cu) (net 28) (status 30))
@@
   (segment (start 165.1 104.14) (end 170.815 98.425) (width 0.3) (layer B.Cu) (net 35))
   (segment (start 156.824058 104.14) (end 165.1 104.14) (width 0.3) (layer B.Cu) (net 35))
-  (segment (start 181.61 95.25) (end 181.61 87.64) (width 0.3) (layer F.Cu) (net 36))
-  (segment (start 181.61 87.64) (end 180.33 86.36) (width 0.3) (layer F.Cu) (net 36))
+  (segment (start 176.53 89.535) (end 179.07 86.995) (width 0.3) (layer F.Cu) (net 36))
+  (segment (start 179.07 86.995) (end 179.07 86.36) (width 0.3) (layer F.Cu) (net 36))
+  (segment (start 181.61 95.25) (end 181.61 94.615) (width 0.3) (layer F.Cu) (net 36))
+  (segment (start 181.61 94.615) (end 176.53 89.535) (width 0.3) (layer F.Cu) (net 36))
   (zone (net 18) (net_name GND) (layer F.Cu) (hatch edge 0.508)
     (connect_pads (clearance 0.4))
